Commit message: Modified the URDF file

File: urdf/robot.urdf (robot description, URDF)
Before this commit: robot Selene, 12 links, 11 joints
Links:
- removed link Feet_Left
- removed link Feet_Right
- added link Foot_Left, mass 0.109031223076226; collision mesh filename=file:///$(find humanoid_robot)/meshes/Foot_Left.STL; visual mesh filename=file:///$(find humanoid_robot)/meshes/Foot_Left.STL
- added link Foot_Right, mass 0.109031283085521; collision mesh filename=file:///$(find humanoid_robot)/meshes/Foot_Right.STL; visual mesh filename=file:///$(find humanoid_robot)/meshes/Foot_Right.STL
- link Calf_Left: mass 0.347244355232965 -> 0.327204793273009
- link Calf_Right: mass 0.347222968435987 -> 0.327294266891114
- link Elbow_Left: mass 0.0827614157852023 -> 0.080679640365444
- link Elbow_Right: mass 0.0827455082429507 -> 0.0806748169693422
- link Head: mass 0.020475566345367 -> 0.0204755663453671
- link Shoulder_Left: mass 0.173961442932148 -> 0.17396156125864
- link Shoulder_Right: mass 0.173956563774839 -> 0.173956267653836
- link Thigh_Left: mass 1.71254429261779 -> 1.71253222820306
- link Thigh_Right: mass 1.71247209269631 -> 1.71249589076309
- link base_link: mass 3.7818 -> 3.78181180876983
Joints:
- removed joint CalfFeet_Left
- removed joint CalfFeet_Right
- added joint CalfFoot_Left: type continuous, parent Calf_Left, child Foot_Left, origin xyz=0.039418 -0.0024472 -0.17177 rpy=0 0 0, axis 0 1 0
- added joint CalfFoot_Right: type continuous, parent Calf_Right, child Foot_Right, origin xyz=0.039418 0.002408 -0.17177 rpy=0 0 0, axis 0 1 0
- joint Neck: origin xyz=-0.14524 -0.037441 0.83602 rpy=0 0 0 -> xyz=-0.044306 0.010853 0.81525 rpy=0 0 0
- joint ShoulderElbow_Left: origin xyz=0.030403 0.00076605 -0.14862 rpy=0 0 0 -> xyz=-0.00073185 -0.040103 -0.14681 rpy=0 0 0
- joint ShoulderElbow_Right: origin xyz=0.030359 -0.00076495 -0.14862 rpy=0 0 0 -> xyz=-0.00073185 0.040103 -0.14681 rpy=0 0 0
- joint ThighCalf_Left: axis 0.0094744 0.99913 -0.040492 -> 0 1 0; origin xyz=0.05817 -0.01741 -0.31668 rpy=0 0 0 -> xyz=0.0094239 -0.039542 -0.32005 rpy=0 0 0
- joint ThighCalf_Right: axis -0.15989 0.98597 -0.047997 -> 0 1 0; origin xyz=0.091715 -0.00051607 -0.31612 rpy=0 0 0 -> xyz=0.0094239 0.039542 -0.32005 rpy=0 0 0
- joint TorsoShoulder_Left: axis -1 0 0 -> 1 0 0; origin xyz=-0.099564 -0.11999 0.79337 rpy=0 0 0 -> xyz=-0.033379 -0.064693 0.78215 rpy=0 0 0
- joint TorsoShoulder_Right: axis -1 0 0 -> 1 0 0; origin xyz=-0.09949 0.043597 0.79036 rpy=0 0 0 -> xyz=-0.033308 0.08489 0.77914 rpy=0 0 0
- joint TorsoThigh_Left: limit lower=-1.0 upper=1.0 effort=10 velocity=5 -> (none); origin xyz=-0.11512 -0.065021 0.55768 rpy=0 0 0 -> xyz=-0.013335 -0.010993 0.55295 rpy=0 0 0
- joint TorsoThigh_Right: axis -1 0 0 -> 1 0 0; origin xyz=-0.11209 -0.0024223 0.55516 rpy=0 0 0 -> xyz=-0.015152 0.040137 0.55044 rpy=0 0 0

Commit message: Added the SDF file

File: urdf/robot.urdf (robot description, URDF)
Before this commit: robot Selene, 12 links, 11 joints
Links:
- added link world
Joints:
- added joint Hang: type fixed, parent world, child base_link
