Commit message: add joint trajectory nodetest to CI

File: urdf/robot.urdf.xacro (robot description, xacro)
@@ -573,250 +573,4 @@
     </plugin>
     <pose>0 0 0 0 0 0</pose>
-    </sensor>
-  </gazebo>
-  <!-- *****************   Force-Torque Sensors on All Joints   ***************** -->
-  <!-- Neck Yaw -->
-  <gazebo reference="Neck_Yaw">
-    <sensor name="force_torque_sensor" type="force_torque">
-      <always_on>true</always_on>
-      <update_rate>100</update_rate>
-      <visualize>true</visualize>
-      <topic>force_torque1</topic>
-      <force_torque>
-        <frame>child</frame>
-        <measure_direction>parent_to_child</measure_direction>
-      </force_torque>
-      <pose>0 0 0 0 0 0</pose>
-    </sensor>
-  </gazebo>
-  <!-- Neck Pitch -->
-  <gazebo reference="Neck_Pitch">
-    <sensor name="force_torque_sensor" type="force_torque">
-      <always_on>true</always_on>
-      <update_rate>100</update_rate>
-      <visualize>true</visualize>
-      <topic>force_torque11</topic>
-      <force_torque>
-        <frame>child</frame>
-        <measure_direction>parent_to_child</measure_direction>
-      </force_torque>
-      <pose>0 0 0 0 0 0</pose>
-    </sensor>
-  </gazebo>
-  <!-- Left Shoulder Pitch -->
-  <gazebo reference="TorsoShoulder_Left_Pitch">
-    <sensor name="force_torque_sensor" type="force_torque">
-      <always_on>true</always_on>
-      <update_rate>100</update_rate>
-      <visualize>true</visualize>
-      <topic>force_torque2</topic>
-      <force_torque>
-        <frame>child</frame>
-        <measure_direction>parent_to_child</measure_direction>
-      </force_torque>
-      <pose>0 0 0 0 0 0</pose>
-    </sensor>
-  </gazebo>
-  <!-- Left Shoulder Roll -->
-  <gazebo reference="TorsoShoulder_Left_Roll">
-    <sensor name="force_torque_sensor" type="force_torque">
-      <always_on>true</always_on>
-      <update_rate>100</update_rate>
-      <visualize>true</visualize>
-      <topic>force_torque22</topic>
-      <force_torque>
-        <frame>child</frame>
-        <measure_direction>parent_to_child</measure_direction>
-      </force_torque>
-      <pose>0 0 0 0 0 0</pose>
-    </sensor>
-  </gazebo>
-  <!-- Left Elbow Pitch -->
-  <gazebo reference="ShoulderElbow_Left">
-    <sensor name="force_torque_sensor" type="force_torque">
-      <always_on>true</always_on>
-      <update_rate>100</update_rate>
-      <visualize>true</visualize>
-      <topic>force_torque3</topic>
-      <force_torque>
-        <frame>child</frame>
-        <measure_direction>parent_to_child</measure_direction>
-      </force_torque>
-      <pose>0 0 0 0 0 0</pose>
-    </sensor>
-  </gazebo>
-  <!-- Right Shoulder Pitch -->
-  <gazebo reference="TorsoShoulder_Right_Pitch">
-    <sensor name="force_torque_sensor" type="force_torque">
-      <always_on>true</always_on>
-      <update_rate>100</update_rate>
-      <visualize>true</visualize>
-      <topic>force_torque2</topic>
-      <force_torque>
-        <frame>child</frame>
-        <measure_direction>parent_to_child</measure_direction>
-      </force_torque>
-      <pose>0 0 0 0 0 0</pose>
-    </sensor>
-  </gazebo>
-  <!-- Right Shoulder Roll -->
-  <gazebo reference="TorsoShoulder_Right_Roll">
-    <sensor name="force_torque_sensor" type="force_torque">
-      <always_on>true</always_on>
-      <update_rate>100</update_rate>
-      <visualize>true</visualize>
-      <topic>force_torque22</topic>
-      <force_torque>
-        <frame>child</frame>
-        <measure_direction>parent_to_child</measure_direction>
-      </force_torque>
-      <pose>0 0 0 0 0 0</pose>
-    </sensor>
-  </gazebo>
-  <!-- Right Elbow Pitch -->
-  <gazebo reference="ShoulderElbow_Right">
-    <sensor name="force_torque_sensor" type="force_torque">
-      <always_on>true</always_on>
-      <update_rate>100</update_rate>
-      <visualize>true</visualize>
-      <topic>force_torque3</topic>
-      <force_torque>
-        <frame>child</frame>
-        <measure_direction>parent_to_child</measure_direction>
-      </force_torque>
-      <pose>0 0 0 0 0 0</pose>
-    </sensor>
-  </gazebo>
-  <!-- Left Thigh Pitch -->
-  <gazebo reference="TorsoThigh_Left_Pitch">
-    <sensor name="force_torque_sensor" type="force_torque">
-      <always_on>true</always_on>
-      <update_rate>100</update_rate>
-      <visualize>true</visualize>
-      <topic>force_torque4</topic>
-      <force_torque>
-        <frame>child</frame>
-        <measure_direction>parent_to_child</measure_direction>
-      </force_torque>
-      <pose>0 0 0 0 0 0</pose>
-    </sensor>
-  </gazebo>
-  <!-- Left Thigh Yaw -->
-  <gazebo reference="TorsoThigh_Left_Yaw">
-    <sensor name="force_torque_sensor" type="force_torque">
-      <always_on>true</always_on>
-      <update_rate>100</update_rate>
-      <visualize>true</visualize>
-      <topic>force_torque44</topic>
-      <force_torque>
-        <frame>child</frame>
-        <measure_direction>parent_to_child</measure_direction>
-      </force_torque>
-      <pose>0 0 0 0 0 0</pose>
-    </sensor>
-  </gazebo>
-   <!-- Left Calf Pitch -->
-  <gazebo reference="ThighCalf_Left">
-    <sensor name="force_torque_sensor" type="force_torque">
-      <always_on>true</always_on>
-      <update_rate>100</update_rate>
-      <visualize>true</visualize>
-      <topic>force_torque5</topic>
-      <force_torque>
-        <frame>child</frame>
-        <measure_direction>parent_to_child</measure_direction>
-      </force_torque>
-      <pose>0 0 0 0 0 0</pose>
-    </sensor>
-  </gazebo>
-  <!-- Left Foot Pitch -->
-  <gazebo reference="CalfFoot_Left">
-    <sensor name="force_torque_sensor" type="force_torque">
-      <always_on>true</always_on>
-      <update_rate>100</update_rate>
-      <visualize>true</visualize>
-      <topic>force_torque6</topic>
-      <force_torque>
-        <frame>child</frame>
-        <measure_direction>parent_to_child</measure_direction>
-      </force_torque>
-      <pose>0 0 0 0 0 0</pose>
-    </sensor>
-  </gazebo>
-  <!-- Right Thigh Pitch -->
-  <gazebo reference="TorsoThigh_Right_Pitch">
-    <sensor name="force_torque_sensor" type="force_torque">
-      <always_on>true</always_on>
-      <update_rate>100</update_rate>
-      <visualize>true</visualize>
-      <topic>force_torque7</topic>
-      <force_torque>
-        <frame>child</frame>
-        <measure_direction>parent_to_child</measure_direction>
-      </force_torque>
-      <pose>0 0 0 0 0 0</pose>
-    </sensor>
-  </gazebo>
-  <!-- Right Thigh Yaw -->
-  <gazebo reference="TorsoThigh_Right_Yaw">
-    <sensor name="force_torque_sensor" type="force_torque">
-      <always_on>true</always_on>
-      <update_rate>100</update_rate>
-      <visualize>true</visualize>
-      <topic>force_torque77</topic>
-      <force_torque>
-        <frame>child</frame>
-        <measure_direction>parent_to_child</measure_direction>
-      </force_torque>
-      <pose>0 0 0 0 0 0</pose>
-    </sensor>
-  </gazebo>
-   <!-- Right Calf Pitch -->
-  <gazebo reference="ThighCalf_Right">
-    <sensor name="force_torque_sensor" type="force_torque">
-      <always_on>true</always_on>
-      <update_rate>100</update_rate>
-      <visualize>true</visualize>
-      <topic>force_torque8</topic>
-      <force_torque>
-        <frame>child</frame>
-        <measure_direction>parent_to_child</measure_direction>
-      </force_torque>
-      <pose>0 0 0 0 0 0</pose>
-    </sensor>
-  </gazebo>
-  <!-- Right Foot Pitch -->
-  <gazebo reference="CalfFoot_Right">
-    <sensor name="force_torque_sensor" type="force_torque">
-      <always_on>true</always_on>
-      <update_rate>100</update_rate>
-      <visualize>true</visualize>
-      <topic>force_torque88</topic>
-      <force_torque>
-        <frame>child</frame>
-        <measure_direction>parent_to_child</measure_direction>
-      </force_torque>
-      <pose>0 0 0 0 0 0</pose>
-    </sensor>
-  </gazebo>
-  <!-- ****************************   Contact Sensors   **************************** -->
-  <gazebo reference="Foot_Right">
-    <sensor name="contact_sensor_right" type="contact">
-      <update_rate>100</update_rate>
-      <always_on>true</always_on>
-      <visualize>true</visualize>
-      <contact>
-        <collision>Foot_Right_collision</collision>
-      </contact>
-    </sensor>
-  </gazebo>
-  <gazebo reference="Foot_Left">
-    <sensor name="contact_sensor_left" type="contact">
-      <update_rate>100</update_rate>
-      <always_on>true</always_on>
-      <visualize>true</visualize>
-      <contact>
-        <collision>Foot_Left_collision</collision>
-      </contact>
     </sensor>
   </gazebo>
