Commit message: add rl env ros2_control issue remains

File: urdf/robot.urdf.xacro (robot description, xacro)
@@ -5,6 +5,6 @@
   <link name="base_link">
     <inertial>
+      <mass value="3.78181180876983" />
       <origin xyz="-0.0100023420943865 0.0113704665181975 0.674727562757712" rpy="0 0 0" />
-      <mass value="3.78181180876983" />
       <inertia
         ixx="0.0289881715545131" ixy="-2.34952842388438E-05" ixz="0.00203838739877037"
@@ -28,6 +28,6 @@
   <link name="Head">
     <inertial>
+      <mass value="0.0204755663453671" />
       <origin xyz="1.94507491572959E-06 -1.10276307547261E-07 0.00920379107702982" rpy="0 0 0" />
-      <mass value="0.0204755663453671" />
       <inertia
         ixx="2.48857313055502E-06" ixy="1.58933146859342E-11" ixz="-1.53587889097411E-11"
@@ -50,9 +50,8 @@
   <link name="Neck_Yaw_Link">
     <inertial>
+      <mass value="0.05"/>
       <origin xyz=" 0 0 0" rpy="0 0 0" />
-      <mass value="0.0001"/>
-      <inertia ixx="1e-6" ixy="0" ixz="0"
-              iyy="1e-6" iyz="0" izz="1e-6"/>
-      </inertial>
+      <inertia ixx="0.001" iyy="0.001" izz="0.001" ixy="0" ixz="0" iyz="0"/>
+    </inertial>
     <visual>
       <origin xyz="0 0 0" rpy="0 0 0" />
@@ -73,6 +72,6 @@
   <link name="LShoulder_Pitch_Link">
     <inertial>
+      <mass value="0.17396156125864" />
       <origin xyz="-0.000226132441242099 -0.0354806783650563 -0.0683015626357323" rpy="0 0 0" />
-      <mass value="0.17396156125864" />
       <inertia
         ixx="0.000290783661604433" ixy="8.53619200375728E-08" ixz="9.28025240172068E-07"
@@ -95,9 +94,8 @@
   <link name="LShoulder_Roll_Link">
     <inertial>
+      <mass value="0.05"/>
       <origin xyz=" 0 0 0" rpy="0 0 0" />
-      <mass value="0.0001"/>
-      <inertia ixx="1e-6" ixy="0" ixz="0"
-              iyy="1e-6" iyz="0" izz="1e-6"/>
-      </inertial>
+      <inertia ixx="0.001" iyy="0.001" izz="0.001" ixy="0" ixz="0" iyz="0"/>
+    </inertial>
     <visual>
       <origin xyz="0 0 0" rpy="0 0 0" />
@@ -117,6 +115,6 @@
   <link name="RShoulder_Pitch_Link">
     <inertial>
+      <mass value="0.173956267653836" />
       <origin xyz="-0.000226503959646872 0.0354809522342639 -0.0683034814503672" rpy="0 0 0" />
-      <mass value="0.173956267653836" />
       <inertia
         ixx="0.000290775822093302" ixy="-8.64319034159634E-08" ixz="9.31069079745632E-07"
@@ -139,9 +137,8 @@
   <link name="RShoulder_Roll_Link">
     <inertial>
+      <mass value="0.05"/>
       <origin xyz=" 0 0 0" rpy="0 0 0" />
-      <mass value="0.0001"/>
-      <inertia ixx="1e-6" ixy="0" ixz="0"
-              iyy="1e-6" iyz="0" izz="1e-6"/>
-      </inertial>
+      <inertia ixx="0.001" iyy="0.001" izz="0.001" ixy="0" ixz="0" iyz="0"/>
+    </inertial>
     <visual>
       <origin xyz="0 0 0" rpy="0 0 0" />
@@ -161,6 +158,6 @@
   <link name="Elbow_Left">
     <inertial>
+      <mass value="0.080679640365444" />
       <origin xyz="0.00928267206313797 -0.00549982222068757 -0.0621529175277214" rpy="0 0 0" />
-      <mass value="0.080679640365444" />
       <inertia
         ixx="0.00010013808132852" ixy="8.50147925817831E-07" ixz="2.1171900411E-05"
@@ -183,6 +180,6 @@
   <link name="Elbow_Right">
     <inertial>
+      <mass value="0.0806748169693422" />
       <origin xyz="0.00928283620034147 0.00549966032962597 -0.0621529115970779" rpy="0 0 0" />
-      <mass value="0.0806748169693422" />
       <inertia
         ixx="0.000100130695775464" ixy="-8.50346985914723E-07" ixz="2.11695824904372E-05"
@@ -207,6 +204,6 @@
   <link name="LThigh_Pitch_Link">
     <inertial>
+      <mass value="1.71253222820306" />
       <origin xyz="0.0232782491490201 -0.0391974149526159 -0.143116335507406" rpy="0 0 0" />
-      <mass value="1.71253222820306" />
       <inertia
         ixx="0.00996674674236712" ixy="-3.24702547387314E-05" ixz="0.000390411340022318"
@@ -229,9 +226,8 @@
   <link name="LThigh_Yaw_Link">
     <inertial>
+      <mass value="0.05"/>
       <origin xyz=" 0 0 0" rpy="0 0 0" />
-      <mass value="0.0001"/>
-      <inertia ixx="1e-6" ixy="0" ixz="0"
-              iyy="1e-6" iyz="0" izz="1e-6"/>
-      </inertial>
+      <inertia ixx="0.001" iyy="0.001" izz="0.001" ixy="0" ixz="0" iyz="0"/>
+    </inertial>
     <visual>
       <origin xyz="0 0 0" rpy="0 0 0" />
@@ -250,6 +246,6 @@
   <link name="RThigh_Pitch_Link">
     <inertial>
+      <mass value="1.71249589076309" />
       <origin xyz="0.0232810333065785 0.0391987879827244 -0.143121811370373" rpy="0 0 0" />
-      <mass value="1.71249589076309" />
       <inertia
         ixx="0.00996720981270455" ixy="3.26594381610291E-05" ixz="0.000390081057293533"
@@ -272,9 +268,8 @@
   <link name="RThigh_Yaw_Link">
     <inertial>
+      <mass value="0.05"/>
       <origin xyz=" 0 0 0" rpy="0 0 0" />
-      <mass value="0.0001"/>
-      <inertia ixx="1e-6" ixy="0" ixz="0"
-              iyy="1e-6" iyz="0" izz="1e-6"/>
-      </inertial>
+      <inertia ixx="0.001" iyy="0.001" izz="0.001" ixy="0" ixz="0" iyz="0"/>
+    </inertial>
     <visual>
       <origin xyz="0 0 0" rpy="0 0 0" />
@@ -294,6 +289,6 @@
   <link name="Calf_Left">
     <inertial>
+      <mass value="0.327204793273009" />
       <origin xyz="0.0190102600468827 -0.00159963895885237 -0.076517992366644" rpy="0 0 0" />
-      <mass value="0.327204793273009" />
       <inertia
         ixx="0.00056060655488805" ixy="1.83941448046734E-06" ixz="0.000117382611516597"
@@ -316,6 +311,6 @@
   <link name="Calf_Right">
     <inertial>
+      <mass value="0.327294266891114" />
       <origin xyz="0.0190029389282548 0.00159876373223955 -0.0765008487844586" rpy="0 0 0" />
-      <mass value="0.327294266891114" />
       <inertia
         ixx="0.000560814729177772" ixy="-1.8532188939462E-06" ixz="0.000117482190032848"
@@ -339,6 +334,6 @@
   <link name="Foot_Left">
     <inertial>
+      <mass value="0.109031223076226" />
       <origin xyz="0.0302743738770081 8.60405123109392E-05 -0.0409960721960091" rpy="0 0 0" />
-      <mass value="0.109031223076226" />
       <inertia
         ixx="3.015596373348E-05" ixy="1.2148890528659E-07" ixz="1.81609695852798E-05"
@@ -361,6 +356,6 @@
   <link name="Foot_Right">
     <inertial>
+      <mass value="0.109031283085521" />
       <origin xyz="0.0302743600707219 8.60381006145966E-05 -0.0409960624720848" rpy="0 0 0" />
-      <mass value="0.109031283085521" />
       <inertia
         ixx="3.01560100675454E-05" ixy="1.21487322311586E-07" ixz="1.81609850738135E-05"
@@ -380,10 +375,5 @@
     </collision>
   </link>
-  <link name="world"/>
-  <!-- #######################################################   JOINTS   ################################################################### -->
-  <joint name="Hang" type="fixed">
-    <parent link="world"/>
-    <child link="base_link"/>
-  </joint>
+  <!-- ##############################################   JOINTS   ################################################ -->
   <!-- Neck -->
   <joint name="Neck_Yaw" type="revolute">
@@ -393,5 +383,5 @@
     <axis xyz="0 0 1" />
     <limit lower="-1.0472" upper="1.0472" effort="1.0" velocity="1.0"/> <!-- 60 degrees-->
-    <dynamics damping="0.05" friction="0.5"/>
+    <dynamics damping="0.2" friction="0.5"/>
   </joint>
   <joint name="Neck_Pitch" type="revolute">
@@ -401,5 +391,5 @@
     <axis xyz="0 1 0" />
     <limit lower="-0.523599" upper="0.523599" effort="1.0" velocity="1.0"/> <!-- 30 degrees -->
-    <dynamics damping="0.05" friction="0.5"/>
+    <dynamics damping="0.2" friction="0.5"/>
   </joint>
   <!-- Left Shoulder and Torso Roll -->
@@ -410,5 +400,5 @@
     <axis xyz="1 0 0" />
     <limit lower="-1.0472" upper="0" effort="1.0" velocity="1.0"/> <!-- 0 - 60 degrees -->
-    <dynamics damping="0.05" friction="0.5"/>
+    <dynamics damping="0.2" friction="0.5"/>
   </joint>
   <!-- Left Shoulder Pitch -->
@@ -419,5 +409,5 @@
     <axis xyz="0 1 0" />
     <limit lower="-3.14159" upper="0.349066" effort="1.0" velocity="1.0"/> <!-- (-20) - 180 degrees-->
-    <dynamics damping="0.05" friction="0.5"/>
+    <dynamics damping="0.2" friction="0.5"/>
   </joint>
   <!-- Left Elbow and Shoulder -->
@@ -428,5 +418,5 @@
     <axis xyz="-0.025189 0.99968 0" />
     <limit lower="-1.74533" upper="0.349066" effort="1.0" velocity="1.0"/> <!-- (-20) - 100 deg-->
-    <dynamics damping="0.05" friction="0.5"/>
+    <dynamics damping="0.2" friction="0.5"/>
   </joint>
   <!-- Right Shoulder and Torso Roll-->
@@ -437,5 +427,5 @@
     <axis xyz="1 0 0" />
     <limit lower="0" upper="1.0472" effort="1.0" velocity="1.0"/> <!-- 0 - 60 degrees -->
-    <dynamics damping="0.05" friction="0.5"/>
+    <dynamics damping="0.2" friction="0.5"/>
   </joint>
   <!-- Right Shoulder Pitch -->
@@ -446,5 +436,5 @@
     <axis xyz="0 1 0" />
     <limit lower="-3.14159" upper="0.349066" effort="1.0" velocity="1.0"/> <!-- (-20) - 180 degrees-->
-    <dynamics damping="0.05" friction="0.5"/>
+    <dynamics damping="0.2" friction="0.5"/>
   </joint>
   <!-- Right Elbow and Shoulder -->
@@ -455,5 +445,5 @@
     <axis xyz="0.025189 0.99968 0" />
     <limit lower="-1.74533" upper="0.349066" effort="1.0" velocity="1.0"/> <!-- (-20) to 100 deg-->
-    <dynamics damping="0.05" friction="0.5"/>
+    <dynamics damping="0.2" friction="0.5"/>
   </joint>
   <!-- Left Thigh and Torso Yaw -->
@@ -464,5 +454,5 @@
     <axis xyz="0 0 1" />
     <limit lower="-0.0872665" upper="0.349066" effort="1.0" velocity="1.0"/> <!-- (-5) - 20 degrees -->
-    <dynamics damping="0.05" friction="0.5"/>
+    <dynamics damping="0.2" friction="0.5"/>
   </joint>
   <!-- Left Thigh and Torso Pitch -->
@@ -473,5 +463,5 @@
     <axis xyz="0 1 0" />
     <limit lower="-2.0944" upper="0.349066" effort="1.0" velocity="1.0"/> <!-- (-60) - 120 degrees-->
-    <dynamics damping="0.05" friction="0.5"/>
+    <dynamics damping="0.2" friction="0.5"/>
   </joint>
   <!-- Left Calf and Thigh -->
@@ -482,5 +472,5 @@
     <axis xyz="0 1 0" />
     <limit lower="-0.349066" upper="1.74533" effort="1.0" velocity="1.0"/> <!-- (-20) - 100 degrees-->
-    <dynamics damping="0.05" friction="0.5"/>
+    <dynamics damping="0.2" friction="0.5"/>
   </joint>
   <!-- Left Foot and Calf -->
@@ -491,5 +481,5 @@
     <axis xyz="0 1 0" />
     <limit lower="-0.785398" upper="0.785398" effort="1.0" velocity="1.0"/> <!-- 45 degrees-->
-    <dynamics damping="0.05" friction="0.5"/>
+    <dynamics damping="0.2" friction="0.5"/>
   </joint>
   <!-- Right Thigh and Torso Yaw -->
@@ -500,5 +490,5 @@
     <axis xyz="0 0 1" />
     <limit lower="-0.0872665" upper="0.349066" effort="1.0" velocity="1.0"/> <!-- (-5) - 20 degrees -->
-    <dynamics damping="0.05" friction="0.5"/>
+    <dynamics damping="0.2" friction="0.5"/>
   </joint>
   <!-- Right Thigh and Torso Pitch -->
@@ -509,5 +499,5 @@
     <axis xyz="0 1 0" />
     <limit lower="-2.0944" upper="0.349066" effort="1.0" velocity="1.0"/> <!-- 60 - (-120) degrees-->
-    <dynamics damping="0.05" friction="0.5"/>
+    <dynamics damping="0.2" friction="0.5"/>
   </joint>
   <!-- Right Calf and Thigh -->
@@ -518,5 +508,5 @@
     <axis xyz="0 1 0" />
     <limit lower="-0.349066" upper="1.74533" effort="1.0" velocity="1.0"/> <!-- (-20) - 100 degrees-->
-    <dynamics damping="0.05" friction="0.5"/>
+    <dynamics damping="0.2" friction="0.5"/>
   </joint>
   <!-- Right Foot and Calf -->
@@ -527,5 +517,5 @@
     <axis xyz="0 1 0" />
     <limit lower="-0.785398" upper="0.785398" effort="1.0" velocity="1.0"/> <!-- 45 degrees-->
-    <dynamics damping="0.05" friction="0.5"/>
+    <dynamics damping="0.2" friction="0.5"/>
   </joint>
   <!-- ****************************   IMU Sensor   **************************** -->
@@ -605,4 +595,5 @@
     <plugin filename="libgazebo_ros2_control.so" name="gazebo_ros2_control">
       <parameters>$(find humanoid_robot)/config/controller_config.yaml</parameters>
+      <hold_joints>false</hold_joints>
     </plugin>
   </gazebo>
@@ -612,80 +603,80 @@
     </hardware>
     <joint name="Neck_Yaw">
-      <command_interface name="position"/>
+      <command_interface name="position_pid"/>
       <state_interface name="position"/>
       <state_interface name="velocity"/>
     </joint>
     <joint name="Neck_Pitch">
-      <command_interface name="position"/>
+      <command_interface name="position_pid"/>
       <state_interface name="position"/>
       <state_interface name="velocity"/>
     </joint>
     <joint name="TorsoShoulder_Left_Pitch">
-      <command_interface name="position"/>
+      <command_interface name="position_pid"/>
       <state_interface name="position"/>
       <state_interface name="velocity"/>
     </joint>
     <joint name="TorsoShoulder_Left_Roll">
-      <command_interface name="position"/>
+      <command_interface name="position_pid"/>
       <state_interface name="position"/>
       <state_interface name="velocity"/>
     </joint>
     <joint name="ShoulderElbow_Left">
-      <command_interface name="position"/>
+      <command_interface name="position_pid"/>
       <state_interface name="position"/>
       <state_interface name="velocity"/>
     </joint>
     <joint name="TorsoShoulder_Right_Pitch">
-      <command_interface name="position"/>
+      <command_interface name="position_pid"/>
       <state_interface name="position"/>
       <state_interface name="velocity"/>
     </joint>
     <joint name="TorsoShoulder_Right_Roll">
-      <command_interface name="position"/>
+      <command_interface name="position_pid"/>
       <state_interface name="position"/>
       <state_interface name="velocity"/>
     </joint>
     <joint name="ShoulderElbow_Right">
-      <command_interface name="position"/>
+      <command_interface name="position_pid"/>
       <state_interface name="position"/>
       <state_interface name="velocity"/>
     </joint>
     <joint name="TorsoThigh_Left_Pitch">
-      <command_interface name="position"/>
+      <command_interface name="position_pid"/>
       <state_interface name="position"/>
       <state_interface name="velocity"/>
     </joint>
     <joint name="TorsoThigh_Left_Yaw">
-      <command_interface name="position"/>
+      <command_interface name="position_pid"/>
       <state_interface name="position"/>
       <state_interface name="velocity"/>
     </joint>
     <joint name="ThighCalf_Left">
-      <command_interface name="position"/>
+      <command_interface name="position_pid"/>
       <state_interface name="position"/>
       <state_interface name="velocity"/>
     </joint>
     <joint name="CalfFoot_Left">
-      <command_interface name="position"/>
+      <command_interface name="position_pid"/>
       <state_interface name="position"/>
       <state_interface name="velocity"/>
     </joint>
     <joint name="TorsoThigh_Right_Pitch">
-      <command_interface name="position"/>
+      <command_interface name="position_pid"/>
       <state_interface name="position"/>
       <state_interface name="velocity"/>
     </joint>
     <joint name="TorsoThigh_Right_Yaw">
-      <command_interface name="position"/>
+      <command_interface name="position_pid"/>
       <state_interface name="position"/>
       <state_interface name="velocity"/>
     </joint>
     <joint name="ThighCalf_Right">
-      <command_interface name="position"/>
+      <command_interface name="position_pid"/>
       <state_interface name="position"/>
       <state_interface name="velocity"/>
     </joint>
     <joint name="CalfFoot_Right">
-      <command_interface name="position"/>
+      <command_interface name="position_pid"/>
       <state_interface name="position"/>
       <state_interface name="velocity"/>
