Commit message: add environment setup code

File: urdf/robot.urdf.xacro (robot description, xacro)
@@ -1,845 +1,7 @@
 <?xml version="1.0"?>
-<robot name="Selene" xmlns:xacro="http://www.ros.org/wiki/xacro">
-  <!-- #######################################################   LINKS   ################################################################### -->
-  <!-- Base -->
-  <link name="base_link">
-    <inertial>
-      <mass value="3.78181180876983" />
-      <origin xyz="-0.0100023420943865 0.0113704665181975 0.674727562757712" rpy="0 0 0" />
-      <inertia
-        ixx="0.0289881715545131" ixy="-2.34952842388438E-05" ixz="0.00203838739877037"
-        iyy="0.0282471940044164" iyz="0.000277812220276223" izz="0.00985571887812677" />
-    </inertial>
-    <visual>
-      <origin xyz="0 0 0" rpy="0 0 0" />
-      <geometry>
-        <mesh filename="$(find humanoid_robot)/meshes/base_link.STL"/>
-      </geometry>
-    </visual>
-    <collision>
-      <origin xyz="0 0 0" rpy="0 0 0" />
-      <geometry>
-        <mesh filename="$(find humanoid_robot)/meshes/base_link.STL"/>
-      </geometry>
-    </collision>
-  </link>
-  <!-- #####  UPPER BODY  ##### -->
-  <!-- Head -->
-  <link name="Head">
-    <inertial>
-      <mass value="0.0204755663453671" />
-      <origin xyz="1.94507491572959E-06 -1.10276307547261E-07 0.00920379107702982" rpy="0 0 0" />
-      <inertia
-        ixx="2.48857313055502E-06" ixy="1.58933146859342E-11" ixz="-1.53587889097411E-11"
-        iyy="2.48861362838572E-06" iyz="1.0524516855652E-12" izz="2.30241709600154E-06" />
-    </inertial>
-    <visual>
-      <origin xyz="0 0 0" rpy="0 0 0" />
-      <geometry>
-        <mesh filename="$(find humanoid_robot)/meshes/Head.STL"/>
-      </geometry>
-    </visual>
-    <collision>
-      <origin xyz="0 0 0" rpy="0 0 0" />
-      <geometry>
-        <mesh filename="$(find humanoid_robot)/meshes/Head.STL"/>
-      </geometry>
-    </collision>
-  </link>
-  <!-- Neck_Yaw -->
-  <link name="Neck_Yaw_Link">
-    <inertial>
-      <mass value="0.05"/>
-      <origin xyz=" 0 0 0" rpy="0 0 0" />
-      <inertia ixx="0.001" iyy="0.001" izz="0.001" ixy="0" ixz="0" iyz="0"/>
-    </inertial>
-    <visual>
-      <origin xyz="0 0 0" rpy="0 0 0" />
-      <geometry>
-        <sphere radius="0.001"/>
-      </geometry>
-    </visual>
-    <collision>
-      <origin xyz="0 0 0" rpy="0 0 0" />
-      <geometry>
-        <sphere radius="0.001"/>
-      </geometry>
-    </collision>
-  </link>
-  <!-- *****  Shoulders  ***** -->
-  <!-- Left Shoulder -->
-  <!-- Left Shoulder Pitch Link -->
-  <link name="LShoulder_Pitch_Link">
-    <inertial>
-      <mass value="0.17396156125864" />
-      <origin xyz="-0.000226132441242099 -0.0354806783650563 -0.0683015626357323" rpy="0 0 0" />
-      <inertia
-        ixx="0.000290783661604433" ixy="8.53619200375728E-08" ixz="9.28025240172068E-07"
-        iyy="0.000299832000761949" iyz="-4.02822461595027E-05" izz="4.9521505630746E-05" />
-    </inertial>
-    <visual>
-      <origin xyz="0 0 0" rpy="0 0 0" />
-      <geometry>
-        <mesh filename="$(find humanoid_robot)/meshes/Shoulder_Left.STL"/>
-      </geometry>
-    </visual>
-    <collision>
-      <origin xyz="0 0 0" rpy="0 0 0" />
-      <geometry>
-        <mesh filename="$(find humanoid_robot)/meshes/Shoulder_Left.STL"/>
-      </geometry>
-    </collision>
-  </link>
-  <!-- Left Shoulder Roll Link -->
-  <link name="LShoulder_Roll_Link">
-    <inertial>
-      <mass value="0.05"/>
-      <origin xyz=" 0 0 0" rpy="0 0 0" />
-      <inertia ixx="0.001" iyy="0.001" izz="0.001" ixy="0" ixz="0" iyz="0"/>
-    </inertial>
-    <visual>
-      <origin xyz="0 0 0" rpy="0 0 0" />
-      <geometry>
-        <sphere radius="0.001"/>
-      </geometry>
-    </visual>
-    <collision>
-      <origin xyz="0 0 0" rpy="0 0 0" />
-      <geometry>
-        <sphere radius="0.001"/>
-      </geometry>
-    </collision>
-  </link>
-  <!-- Right Shoulder -->
-  <!-- Right Shoulder Pitch Link -->
-  <link name="RShoulder_Pitch_Link">
-    <inertial>
-      <mass value="0.173956267653836" />
-      <origin xyz="-0.000226503959646872 0.0354809522342639 -0.0683034814503672" rpy="0 0 0" />
-      <inertia
-        ixx="0.000290775822093302" ixy="-8.64319034159634E-08" ixz="9.31069079745632E-07"
-        iyy="0.000299820943485111" iyz="4.02820062142174E-05" izz="4.95193455301138E-05" />
-    </inertial>
-    <visual>
-      <origin xyz="0 0 0" rpy="0 0 0" />
-      <geometry>
-        <mesh filename="$(find humanoid_robot)/meshes/Shoulder_Right.STL"/>
-      </geometry>
-    </visual>
-    <collision>
-      <origin xyz="0 0 0" rpy="0 0 0" />
-      <geometry>
-        <mesh filename="$(find humanoid_robot)/meshes/Shoulder_Right.STL"/>
-      </geometry>
-    </collision>
-  </link>
-  <!-- Right Shoulder Roll Link -->
-  <link name="RShoulder_Roll_Link">
-    <inertial>
-      <mass value="0.05"/>
-      <origin xyz=" 0 0 0" rpy="0 0 0" />
-      <inertia ixx="0.001" iyy="0.001" izz="0.001" ixy="0" ixz="0" iyz="0"/>
-    </inertial>
-    <visual>
-      <origin xyz="0 0 0" rpy="0 0 0" />
-      <geometry>
-        <sphere radius="0.001"/>
-      </geometry>
-    </visual>
-    <collision>
-      <origin xyz="0 0 0" rpy="0 0 0" />
-      <geometry>
-        <sphere radius="0.001"/>
-      </geometry>
-    </collision>
-  </link>
-  <!-- *****  Elbows  ***** -->
-  <!-- Left Elbow -->
-  <link name="Elbow_Left">
-    <inertial>
-      <mass value="0.080679640365444" />
-      <origin xyz="0.00928267206313797 -0.00549982222068757 -0.0621529175277214" rpy="0 0 0" />
-      <inertia
-        ixx="0.00010013808132852" ixy="8.50147925817831E-07" ixz="2.1171900411E-05"
-        iyy="0.000104805954367755" iyz="-4.722322383949E-06" izz="1.42978234327262E-05" />
-    </inertial>
-    <visual>
-      <origin xyz="0 0 0" rpy="0 0 0" />
-      <geometry>
-        <mesh filename="$(find humanoid_robot)/meshes/Elbow_Left.STL"/>
-      </geometry>
-    </visual>
-    <collision>
-      <origin xyz="0 0 0" rpy="0 0 0" />
-      <geometry>
-        <mesh filename="$(find humanoid_robot)/meshes/Elbow_Left.STL"/>
-      </geometry>
-    </collision>
-  </link>
-  <!-- Right Elbow -->
-  <link name="Elbow_Right">
-    <inertial>
-      <mass value="0.0806748169693422" />
-      <origin xyz="0.00928283620034147 0.00549966032962597 -0.0621529115970779" rpy="0 0 0" />
-      <inertia
-        ixx="0.000100130695775464" ixy="-8.50346985914723E-07" ixz="2.11695824904372E-05"
-        iyy="0.000104798052557367" iyz="4.7228265405251E-06" izz="1.42969053841886E-05" />
-    </inertial>
-    <visual>
-      <origin xyz="0 0 0" rpy="0 0 0" />
-      <geometry>
-        <mesh filename="$(find humanoid_robot)/meshes/Elbow_Right.STL"/>
-      </geometry>
-    </visual>
-    <collision>
-      <origin xyz="0 0 0" rpy="0 0 0" />
-      <geometry>
-        <mesh filename="$(find humanoid_robot)/meshes/Elbow_Right.STL"/>
-      </geometry>
-    </collision>
-  </link>
-  <!-- #####  UPPER BODY  ##### -->
-  <!-- *****  Thighs  ***** -->
-  <!-- Left Thigh Pitch -->
-  <link name="LThigh_Pitch_Link">
-    <inertial>
-      <mass value="1.71253222820306" />
-      <origin xyz="0.0232782491490201 -0.0391974149526159 -0.143116335507406" rpy="0 0 0" />
-      <inertia
-        ixx="0.00996674674236712" ixy="-3.24702547387314E-05" ixz="0.000390411340022318"
-        iyy="0.00993892919291852" iyz="-0.000169586324129286" izz="0.00203984834862235" />
-    </inertial>
-    <visual>
-      <origin xyz="0 0 0" rpy="0 0 0" />
-      <geometry>
-        <mesh filename="$(find humanoid_robot)/meshes/Thigh_Left.STL"/>
-      </geometry>
-    </visual>
-    <collision>
-      <origin xyz="0 0 0" rpy="0 0 0" />
-      <geometry>
-        <mesh filename="$(find humanoid_robot)/meshes/Thigh_Left.STL"/>
-      </geometry>
-    </collision>
-  </link>
-  <!-- Left Thigh Yaw -->
-  <link name="LThigh_Yaw_Link">
-    <inertial>
-      <mass value="0.05"/>
-      <origin xyz=" 0 0 0" rpy="0 0 0" />
-      <inertia ixx="0.001" iyy="0.001" izz="0.001" ixy="0" ixz="0" iyz="0"/>
-    </inertial>
-    <visual>
-      <origin xyz="0 0 0" rpy="0 0 0" />
-      <geometry>
-        <sphere radius="0.001"/>
-      </geometry>
-    </visual>
-    <collision>
-      <origin xyz="0 0 0" rpy="0 0 0" />
-      <geometry>
-        <sphere radius="0.001"/>
-      </geometry>
-    </collision>
-  </link>
-  <!-- Right Thigh Pitch-->
-  <link name="RThigh_Pitch_Link">
-    <inertial>
-      <mass value="1.71249589076309" />
-      <origin xyz="0.0232810333065785 0.0391987879827244 -0.143121811370373" rpy="0 0 0" />
-      <inertia
-        ixx="0.00996720981270455" ixy="3.26594381610291E-05" ixz="0.000390081057293533"
-        iyy="0.00993943224089701" iyz="0.000169678146787137" izz="0.00204017135515511" />
-    </inertial>
-    <visual>
-      <origin xyz="0 0 0" rpy="0 0 0" />
-      <geometry>
-        <mesh filename="$(find humanoid_robot)/meshes/Thigh_Right.STL"/>
-      </geometry>
-    </visual>
-    <collision>
-      <origin xyz="0 0 0" rpy="0 0 0" />
-      <geometry>
-        <mesh filename="$(find humanoid_robot)/meshes/Thigh_Right.STL"/>
-      </geometry>
-    </collision>
-  </link>
-  <!-- Right Thigh Yaw -->
-  <link name="RThigh_Yaw_Link">
-    <inertial>
-      <mass value="0.05"/>
-      <origin xyz=" 0 0 0" rpy="0 0 0" />
-      <inertia ixx="0.001" iyy="0.001" izz="0.001" ixy="0" ixz="0" iyz="0"/>
-    </inertial>
-    <visual>
-      <origin xyz="0 0 0" rpy="0 0 0" />
-      <geometry>
-        <sphere radius="0.001"/>
-      </geometry>
-    </visual>
-    <collision>
-      <origin xyz="0 0 0" rpy="0 0 0" />
-      <geometry>
-        <sphere radius="0.001"/>
-      </geometry>
-    </collision>
-  </link>
-  <!-- *****  Calves  ***** -->
-  <!-- Left Calf -->
-  <link name="Calf_Left">
-    <inertial>
-      <mass value="0.327204793273009" />
-      <origin xyz="0.0190102600468827 -0.00159963895885237 -0.076517992366644" rpy="0 0 0" />
-      <inertia
-        ixx="0.00056060655488805" ixy="1.83941448046734E-06" ixz="0.000117382611516597"
-        iyy="0.000576927261299078" iyz="-6.31475075527301E-06" izz="0.00015087656827053" />
-    </inertial>
-    <visual>
-      <origin xyz="0 0 0" rpy="0 0 0" />
-      <geometry>
-        <mesh filename="$(find humanoid_robot)/meshes/Calf_Left.STL"/>
-      </geometry>
-    </visual>
-    <collision>
-      <origin xyz="0 0 0" rpy="0 0 0" />
-      <geometry>
-        <mesh filename="$(find humanoid_robot)/meshes/Calf_Left.STL"/>
-      </geometry>
-    </collision>
-  </link>
-  <!-- Right Calf -->
-  <link name="Calf_Right">
-    <inertial>
-      <mass value="0.327294266891114" />
-      <origin xyz="0.0190029389282548 0.00159876373223955 -0.0765008487844586" rpy="0 0 0" />
-      <inertia
-        ixx="0.000560814729177772" ixy="-1.8532188939462E-06" ixz="0.000117482190032848"
-        iyy="0.0005771798350897" iyz="6.35212960050734E-06" izz="0.000150937009047011" />
-    </inertial>
-    <visual>
-      <origin xyz="0 0 0" rpy="0 0 0" />
-      <geometry>
-        <mesh filename="$(find humanoid_robot)/meshes/Calf_Right.STL" />
-      </geometry>
-    </visual>
-    <collision>
-      <origin xyz="0 0 0" rpy="0 0 0" />
-      <geometry>
-        <mesh filename="$(find humanoid_robot)/meshes/Calf_Right.STL" />
-      </geometry>
-    </collision>
-  </link>
-  <!-- *****  Feet  ***** -->
-  <!-- Left Foot -->
-  <link name="Foot_Left">
-    <inertial>
-      <mass value="0.109031223076226" />
-      <origin xyz="0.0302743738770081 8.60405123109392E-05 -0.0409960721960091" rpy="0 0 0" />
-      <inertia
-        ixx="3.015596373348E-05" ixy="1.2148890528659E-07" ixz="1.81609695852798E-05"
-        iyy="9.62099140376856E-05" iyz="-1.16818324795965E-07" izz="8.50912025243183E-05" />
-    </inertial>
-    <visual>
-      <origin xyz="0 0 0" rpy="0 0 0" />
-      <geometry>
-        <mesh filename="$(find humanoid_robot)/meshes/Foot_Left.STL" />
-      </geometry>
-    </visual>
-    <collision>
-      <origin xyz="0 0 0" rpy="0 0 0" />
-      <geometry>
-        <mesh filename="$(find humanoid_robot)/meshes/Foot_Left.STL" />
-      </geometry>
-    </collision>
-  </link>
-  <!-- Right Foot -->
-  <link name="Foot_Right">
-    <inertial>
-      <mass value="0.109031283085521" />
-      <origin xyz="0.0302743600707219 8.60381006145966E-05 -0.0409960624720848" rpy="0 0 0" />
-      <inertia
-        ixx="3.01560100675454E-05" ixy="1.21487322311586E-07" ixz="1.81609850738135E-05"
-        iyy="9.62099859924235E-05" iyz="-1.16800691255442E-07" izz="8.50912377824343E-05" />
-    </inertial>
-    <visual>
-      <origin xyz="0 0 0" rpy="0 0 0" />
-      <geometry>
-        <mesh filename="$(find humanoid_robot)/meshes/Foot_Right.STL" />
-      </geometry>
-    </visual>
-    <collision>
-      <origin xyz="0 0 0" rpy="0 0 0" />
-      <geometry>
-        <mesh filename="$(find humanoid_robot)/meshes/Foot_Right.STL" />
-      </geometry>
-    </collision>
-  </link>
-  <!-- ##############################################   JOINTS   ################################################ -->
-  <!-- Neck -->
-  <joint name="Neck_Yaw" type="revolute">
-    <origin xyz="-0.044306 0.010853 0.81525" rpy="0 0 0" />
-    <parent link="base_link" />
-    <child link="Neck_Yaw_Link" />
-    <axis xyz="0 0 1" />
-    <limit lower="-1.0472" upper="1.0472" effort="1.0" velocity="1.0"/> <!-- 60 degrees-->
-    <dynamics damping="0.2" friction="0.5"/>
-  </joint>
-  <joint name="Neck_Pitch" type="revolute">
-    <origin xyz="0 0 0" rpy="0 0 0" />
-    <parent link="Neck_Yaw_Link" />
-    <child link="Head" />
-    <axis xyz="0 1 0" />
-    <limit lower="-0.523599" upper="0.523599" effort="1.0" velocity="1.0"/> <!-- 30 degrees -->
-    <dynamics damping="0.2" friction="0.5"/>
-  </joint>
-  <!-- Left Shoulder and Torso Roll -->
-  <joint name="TorsoShoulder_Left_Roll" type="revolute">
-    <origin xyz="-0.033379 -0.064693 0.78215" rpy="0 0 0" />
-    <parent link="base_link" />
-    <child link="LShoulder_Roll_Link" />
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