Commit message: refocus to fixed-base upper body control

File: urdf/robot_core.urdf.xacro (robot description, xacro)
@@ -322,10 +322,10 @@
             </geometry>
         </visual>
-        <collision>
+        <!-- <collision>
             <origin xyz="0 0 0" rpy="0 0 0" />
             <geometry>
                 <mesh filename="$(find humanoid_robot)/meshes/Foot_Left.STL" />
             </geometry>
-        </collision>
+        </collision> -->
         </link>
         <link name="Foot_Right">
@@ -343,10 +343,10 @@
             </geometry>
         </visual>
-        <collision>
+        <!-- <collision>
             <origin xyz="0 0 0" rpy="0 0 0" />
             <geometry>
                 <mesh filename="$(find humanoid_robot)/meshes/Foot_Right.STL" />
             </geometry>
-        </collision>
+        </collision> -->
         </link>
         <!-- ****************************   Joints   **************************** -->
@@ -387,7 +387,7 @@
             <parent link="LShoulder_Pitch_Link" />
             <child link="Elbow_Left" />
-            <axis xyz="-0.025189 0.99968 0" />
+            <axis xyz="0 1 0" />
             <limit lower="-1.74533" upper="0.349066" effort="1.0" velocity="1.0"/> <!-- (-20) - 100 deg-->
-            <dynamics damping="0.2" friction="0.5"/>
+            <dynamics damping="0.15" friction="0.2"/>
         </joint>
         <joint name="TorsoShoulder_Right_Roll" type="revolute">
@@ -411,7 +411,7 @@
             <parent link="RShoulder_Pitch_Link" />
             <child link="Elbow_Right" />
-            <axis xyz="0.025189 0.99968 0" />
+            <axis xyz="0 1 0" />
             <limit lower="-1.74533" upper="0.349066" effort="1.0" velocity="1.0"/> <!-- (-20) to 100 deg-->
-            <dynamics damping="0.2" friction="0.5"/>
+            <dynamics damping="0.15" friction="0.2"/>
         </joint>
         <joint name="TorsoThigh_Left_Yaw" type="revolute">
@@ -506,4 +506,7 @@
             <origin xyz="0 0.01 0.6" rpy="0 0 0"/>
         </joint>
+        <gazebo>
+            <plugin name="fixed_base_support" filename="libfixed_base_support_plugin.so"/>
+        </gazebo>
     </xacro:macro>
 </robot>

Commit message: Add stereo eye cameras and cube test object

File: urdf/robot_core.urdf.xacro (robot description, xacro)
@@ -506,6 +506,64 @@
             <origin xyz="0 0.01 0.6" rpy="0 0 0"/>
         </joint>
-        <gazebo>
-            <plugin name="fixed_base_support" filename="libfixed_base_support_plugin.so"/>
+        <!-- ****************************   Camera   **************************** -->
+        <!-- Camera Link -->
+        <link name="eye_left_link">
+        <inertial>
+            <mass value="0.01"/>
+            <origin xyz="0 0 0"/>
+            <inertia ixx="1e-6" ixy="0" ixz="0"
+                    iyy="1e-6" iyz="0"
+                    izz="1e-6"/>
+        </inertial>
+        <visual>
+            <geometry>
+                <sphere radius="0.003"/>
+            </geometry>
+            <origin xyz="0 0 0"/>
+        </visual>
+        <collision>
+            <geometry>
+                <sphere radius="0.003"/>
+            </geometry>
+            <origin xyz="0 0 0"/>
+        </collision>
+        </link>
+        <link name="eye_right_link">
+        <inertial>
+            <mass value="0.01"/>
+            <origin xyz="0 0 0"/>
+            <inertia ixx="1e-6" ixy="0" ixz="0"
+                    iyy="1e-6" iyz="0"
+                    izz="1e-6"/>
+        </inertial>
+        <visual>
+            <geometry>
+                <sphere radius="0.003"/>
+            </geometry>
+            <origin xyz="0 0 0"/>
+        </visual>
+        <collision>
+            <geometry>
+                <sphere radius="0.003"/>
+            </geometry>
+            <origin xyz="0 0 0"/>
+        </collision>
+        </link>
+        <!-- Camera Joint -->
+        <joint name="left_camera_joint" type="fixed">
+            <parent link="Head"/>
+            <child link="eye_left_link"/>
+            <origin xyz="0.035 -0.018 0.077" rpy="0 0 0"/>
+        </joint>
+        <joint name="right_camera_joint" type="fixed">
+            <parent link="Head"/>
+            <child link="eye_right_link"/>
+            <origin xyz="0.035 0.018 0.077" rpy="0 0 0"/>
+        </joint>
+        <gazebo reference="eye_left_link">
+            <material>Gazebo/Grey</material>
+        </gazebo>
+        <gazebo reference="eye_right_link">
+            <material>Gazebo/Grey</material>
         </gazebo>
     </xacro:macro>

File: urdf/ros2_control.xacro (robot description, xacro)
@@ -120,10 +120,10 @@
       </plugin>
     </gazebo>
-    <!-- ****************************   Joint States   **************************** -->
+    <!-- ****************************   IMU Sensor   **************************** -->
     <!-- IMU Ouput Definition -->
     <gazebo reference="imu_link">
         <gravity>true</gravity>
         <sensor name="imu_sensor" type="imu">
-        <always_on>true</always_on>
+        <always_on>false</always_on>
         <update_rate>100</update_rate>
         <visualize>true</visualize>
@@ -140,4 +140,59 @@
         </sensor>
     </gazebo>
+    <!-- Camera Plugin -->
+    <gazebo reference="eye_left_link">
+      <sensor name="left_eye_camera" type="camera">
+      <always_on>true</always_on>
+      <update_rate>15</update_rate>
+      <visualize>true</visualize>
+      <camera>
+      <horizontal_fov>1.047</horizontal_fov>
+      <image>
+          <width>320</width>
+          <height>240</height>
+          <format>R8G8B8</format>
+      </image>
+      <clip>
+          <near>0.05</near>
+          <far>10</far>
+      </clip>
+      </camera>
+      <plugin name="gazebo_ros_camera_left" filename="libgazebo_ros_camera.so">
+          <camera_name>eye_left</camera_name>
+          <image_topic_name>image_raw</image_topic_name>
+          <camera_info_topic_name>camera_info</camera_info_topic_name>
+          <frame_name>eye_left_link</frame_name>
+      </plugin>
+      </sensor>
+    </gazebo>
+    <gazebo reference="eye_right_link">
+      <sensor name="right_eye_camera" type="camera">
+      <always_on>true</always_on>
+      <update_rate>15</update_rate>
+      <visualize>true</visualize>
+      <camera>
+      <horizontal_fov>1.047</horizontal_fov>
+      <image>
+          <width>320</width>
+          <height>240</height>
+          <format>R8G8B8</format>
+      </image>
+      <clip>
+          <near>0.05</near>
+          <far>10</far>
+      </clip>
+      </camera>
+      <plugin name="gazebo_ros_camera_right" filename="libgazebo_ros_camera.so">
+          <camera_name>eye_right</camera_name>
+          <image_topic_name>image_raw</image_topic_name>
+          <camera_info_topic_name>camera_info</camera_info_topic_name>
+          <frame_name>eye_right_link</frame_name>
+      </plugin>
+      </sensor>
+    </gazebo>
+    <!-- Fixed Base Plugin -->
+    <gazebo>
+        <plugin name="fixed_base_support" filename="libfixed_base_support_plugin.so"/>
+    </gazebo>
   </xacro:macro>
 </robot>

Commit message: add basic pick and place functionality

File: urdf/robot_core.urdf.xacro (robot description, xacro)
@@ -14,11 +14,11 @@
             <origin xyz="0 0 0" rpy="0 0 0" />
             <geometry>
-                <mesh filename="$(find humanoid_robot)/meshes/base_link.STL"/>
-            </geometry>
-        </visual>
-        <collision>
-            <origin xyz="0 0 0" rpy="0 0 0" />
-            <geometry>
-                <mesh filename="$(find humanoid_robot)/meshes/base_link.STL"/>
+                <mesh filename="file://$(find humanoid_robot)/meshes/base_link.STL"/>
+            </geometry>
+        </visual>
+        <collision>
+            <origin xyz="0 0 0" rpy="0 0 0" />
+            <geometry>
+                <mesh filename="file://$(find humanoid_robot)/meshes/base_link.STL"/>
             </geometry>
         </collision>
@@ -35,11 +35,11 @@
             <origin xyz="0 0 0" rpy="0 0 0" />
             <geometry>
-                <mesh filename="$(find humanoid_robot)/meshes/Head.STL"/>
-            </geometry>
-        </visual>
-        <collision>
-            <origin xyz="0 0 0" rpy="0 0 0" />
-            <geometry>
-                <mesh filename="$(find humanoid_robot)/meshes/Head.STL"/>
+                <mesh filename="file://$(find humanoid_robot)/meshes/Head.STL"/>
+            </geometry>
+        </visual>
+        <collision>
+            <origin xyz="0 0 0" rpy="0 0 0" />
+            <geometry>
+                <mesh filename="file://$(find humanoid_robot)/meshes/Head.STL"/>
             </geometry>
         </collision>
@@ -75,11 +75,11 @@
             <origin xyz="0 0 0" rpy="0 0 0" />
             <geometry>
-                <mesh filename="$(find humanoid_robot)/meshes/Shoulder_Left.STL"/>
-            </geometry>
-        </visual>
-        <collision>
-            <origin xyz="0 0 0" rpy="0 0 0" />
-            <geometry>
-                <mesh filename="$(find humanoid_robot)/meshes/Shoulder_Left.STL"/>
+                <mesh filename="file://$(find humanoid_robot)/meshes/Shoulder_Left.STL"/>
+            </geometry>
+        </visual>
+        <collision>
+            <origin xyz="0 0 0" rpy="0 0 0" />
+            <geometry>
+                <mesh filename="file://$(find humanoid_robot)/meshes/Shoulder_Left.STL"/>
             </geometry>
         </collision>
@@ -115,11 +115,11 @@
             <origin xyz="0 0 0" rpy="0 0 0" />
             <geometry>
-                <mesh filename="$(find humanoid_robot)/meshes/Shoulder_Right.STL"/>
-            </geometry>
-        </visual>
-        <collision>
-            <origin xyz="0 0 0" rpy="0 0 0" />
-            <geometry>
-                <mesh filename="$(find humanoid_robot)/meshes/Shoulder_Right.STL"/>
+                <mesh filename="file://$(find humanoid_robot)/meshes/Shoulder_Right.STL"/>
+            </geometry>
+        </visual>
+        <collision>
+            <origin xyz="0 0 0" rpy="0 0 0" />
+            <geometry>
+                <mesh filename="file://$(find humanoid_robot)/meshes/Shoulder_Right.STL"/>
             </geometry>
         </collision>
@@ -155,11 +155,11 @@
             <origin xyz="0 0 0" rpy="0 0 0" />
             <geometry>
-                <mesh filename="$(find humanoid_robot)/meshes/Elbow_Left.STL"/>
-            </geometry>
-        </visual>
-        <collision>
-            <origin xyz="0 0 0" rpy="0 0 0" />
-            <geometry>
-                <mesh filename="$(find humanoid_robot)/meshes/Elbow_Left.STL"/>
+                <mesh filename="file://$(find humanoid_robot)/meshes/Elbow_Left.STL"/>
+            </geometry>
+        </visual>
+        <collision>
+            <origin xyz="0 0 0" rpy="0 0 0" />
+            <geometry>
+                <mesh filename="file://$(find humanoid_robot)/meshes/Elbow_Left.STL"/>
             </geometry>
         </collision>
@@ -176,36 +176,15 @@
             <origin xyz="0 0 0" rpy="0 0 0" />
             <geometry>
-                <mesh filename="$(find humanoid_robot)/meshes/Elbow_Right.STL"/>
-            </geometry>
-        </visual>
-        <collision>
-            <origin xyz="0 0 0" rpy="0 0 0" />
-            <geometry>
-                <mesh filename="$(find humanoid_robot)/meshes/Elbow_Right.STL"/>
-            </geometry>
-        </collision>
-        </link>
-        <link name="LThigh_Pitch_Link">
-        <inertial>
-            <mass value="1.71253222820306" />
-            <origin xyz="0.0232782491490201 -0.0391974149526159 -0.143116335507406" rpy="0 0 0" />
-            <inertia
-            ixx="0.00996674674236712" ixy="-3.24702547387314E-05" ixz="0.000390411340022318"
-            iyy="0.00993892919291852" iyz="-0.000169586324129286" izz="0.00203984834862235" />
-        </inertial>
-        <visual>
-            <origin xyz="0 0 0" rpy="0 0 0" />
-            <geometry>
-                <mesh filename="$(find humanoid_robot)/meshes/Thigh_Left.STL"/>
-            </geometry>
-        </visual>
-        <collision>
-            <origin xyz="0 0 0" rpy="0 0 0" />
-            <geometry>
-                <mesh filename="$(find humanoid_robot)/meshes/Thigh_Left.STL"/>
-            </geometry>
-        </collision>
-        </link>
-        <link name="LThigh_Yaw_Link">
+                <mesh filename="file://$(find humanoid_robot)/meshes/Elbow_Right.STL"/>
+            </geometry>
+        </visual>
+        <collision>
+            <origin xyz="0 0 0" rpy="0 0 0" />
+            <geometry>
+                <mesh filename="file://$(find humanoid_robot)/meshes/Elbow_Right.STL"/>
+            </geometry>
+        </collision>
+        </link>
+        <link name="Palm_Left">
         <inertial>
             <mass value="0.05"/>
@@ -226,26 +205,5 @@
         </collision>
         </link>
-        <link name="RThigh_Pitch_Link">
-        <inertial>
-            <mass value="1.71249589076309" />
-            <origin xyz="0.0232810333065785 0.0391987879827244 -0.143121811370373" rpy="0 0 0" />
-            <inertia
-            ixx="0.00996720981270455" ixy="3.26594381610291E-05" ixz="0.000390081057293533"
-            iyy="0.00993943224089701" iyz="0.000169678146787137" izz="0.00204017135515511" />
-        </inertial>
-        <visual>
-            <origin xyz="0 0 0" rpy="0 0 0" />
-            <geometry>
-                <mesh filename="$(find humanoid_robot)/meshes/Thigh_Right.STL"/>
-            </geometry>
-        </visual>
-        <collision>
-            <origin xyz="0 0 0" rpy="0 0 0" />
-            <geometry>
-                <mesh filename="$(find humanoid_robot)/meshes/Thigh_Right.STL"/>
-            </geometry>
-        </collision>
-        </link>
-        <link name="RThigh_Yaw_Link">
+        <link name="Palm_Right">
         <inertial>
             <mass value="0.05"/>
@@ -266,4 +224,84 @@
         </collision>
         </link>
+        <link name="LThigh_Pitch_Link">
+        <inertial>
+            <mass value="1.71253222820306" />
+            <origin xyz="0.0232782491490201 -0.0391974149526159 -0.143116335507406" rpy="0 0 0" />
+            <inertia
+            ixx="0.00996674674236712" ixy="-3.24702547387314E-05" ixz="0.000390411340022318"
+            iyy="0.00993892919291852" iyz="-0.000169586324129286" izz="0.00203984834862235" />
+        </inertial>
+        <visual>
+            <origin xyz="0 0 0" rpy="0 0 0" />
+            <geometry>
+                <mesh filename="file://$(find humanoid_robot)/meshes/Thigh_Left.STL"/>
+            </geometry>
+        </visual>
+        <collision>
+            <origin xyz="0 0 0" rpy="0 0 0" />
+            <geometry>
+                <mesh filename="file://$(find humanoid_robot)/meshes/Thigh_Left.STL"/>
+            </geometry>
+        </collision>
+        </link>
+        <link name="LThigh_Yaw_Link">
+        <inertial>
+            <mass value="0.05"/>
+            <origin xyz=" 0 0 0" rpy="0 0 0" />
+            <inertia ixx="0.001" iyy="0.001" izz="0.001" ixy="0" ixz="0" iyz="0"/>
+        </inertial>
+        <visual>
+            <origin xyz="0 0 0" rpy="0 0 0" />
+            <geometry>
+                <sphere radius="0.001"/>
+            </geometry>
+        </visual>
+        <collision>
+            <origin xyz="0 0 0" rpy="0 0 0" />
+            <geometry>
+                <sphere radius="0.001"/>
+            </geometry>
+        </collision>
+        </link>
+        <link name="RThigh_Pitch_Link">
+        <inertial>
+            <mass value="1.71249589076309" />
+            <origin xyz="0.0232810333065785 0.0391987879827244 -0.143121811370373" rpy="0 0 0" />
+            <inertia
+            ixx="0.00996720981270455" ixy="3.26594381610291E-05" ixz="0.000390081057293533"
+            iyy="0.00993943224089701" iyz="0.000169678146787137" izz="0.00204017135515511" />
+        </inertial>
+        <visual>
+            <origin xyz="0 0 0" rpy="0 0 0" />
+            <geometry>
+                <mesh filename="file://$(find humanoid_robot)/meshes/Thigh_Right.STL"/>
+            </geometry>
+        </visual>
+        <collision>
+            <origin xyz="0 0 0" rpy="0 0 0" />
+            <geometry>
+                <mesh filename="file://$(find humanoid_robot)/meshes/Thigh_Right.STL"/>
+            </geometry>
+        </collision>
+        </link>
+        <link name="RThigh_Yaw_Link">
+        <inertial>
+            <mass value="0.05"/>
+            <origin xyz=" 0 0 0" rpy="0 0 0" />
+            <inertia ixx="0.001" iyy="0.001" izz="0.001" ixy="0" ixz="0" iyz="0"/>
+        </inertial>
+        <visual>
+            <origin xyz="0 0 0" rpy="0 0 0" />
+            <geometry>
+                <sphere radius="0.001"/>
+            </geometry>
+        </visual>
+        <collision>
+            <origin xyz="0 0 0" rpy="0 0 0" />
+            <geometry>
+                <sphere radius="0.001"/>
+            </geometry>
+        </collision>
+        </link>
         <link name="Calf_Left">
         <inertial>
@@ -277,11 +315,11 @@
             <origin xyz="0 0 0" rpy="0 0 0" />
             <geometry>
-                <mesh filename="$(find humanoid_robot)/meshes/Calf_Left.STL"/>
-            </geometry>
-        </visual>
-        <collision>
-            <origin xyz="0 0 0" rpy="0 0 0" />
-            <geometry>
-                <mesh filename="$(find humanoid_robot)/meshes/Calf_Left.STL"/>
+                <mesh filename="file://$(find humanoid_robot)/meshes/Calf_Left.STL"/>
+            </geometry>
+        </visual>
+        <collision>
+            <origin xyz="0 0 0" rpy="0 0 0" />
+            <geometry>
+                <mesh filename="file://$(find humanoid_robot)/meshes/Calf_Left.STL"/>
             </geometry>
         </collision>
@@ -298,11 +336,11 @@
             <origin xyz="0 0 0" rpy="0 0 0" />
             <geometry>
-                <mesh filename="$(find humanoid_robot)/meshes/Calf_Right.STL" />
-            </geometry>
-        </visual>
-        <collision>
-            <origin xyz="0 0 0" rpy="0 0 0" />
-            <geometry>
-                <mesh filename="$(find humanoid_robot)/meshes/Calf_Right.STL" />
+                <mesh filename="file://$(find humanoid_robot)/meshes/Calf_Right.STL" />
+            </geometry>
+        </visual>
+        <collision>
+            <origin xyz="0 0 0" rpy="0 0 0" />
+            <geometry>
+                <mesh filename="file://$(find humanoid_robot)/meshes/Calf_Right.STL" />
             </geometry>
         </collision>
@@ -319,13 +357,13 @@
             <origin xyz="0 0 0" rpy="0 0 0" />
             <geometry>
-                <mesh filename="$(find humanoid_robot)/meshes/Foot_Left.STL" />
-            </geometry>
-        </visual>
-        <!-- <collision>
-            <origin xyz="0 0 0" rpy="0 0 0" />
-            <geometry>
-                <mesh filename="$(find humanoid_robot)/meshes/Foot_Left.STL" />
-            </geometry>
-        </collision> -->
+                <mesh filename="file://$(find humanoid_robot)/meshes/Foot_Left.STL" />
+            </geometry>
+        </visual>
+        <collision>
+            <origin xyz="0 0 0" rpy="0 0 0" />
+            <geometry>
+                <mesh filename="file://$(find humanoid_robot)/meshes/Foot_Left.STL" />
+            </geometry>
+        </collision>
         </link>
         <link name="Foot_Right">
@@ -340,13 +378,13 @@
             <origin xyz="0 0 0" rpy="0 0 0" />
             <geometry>
-                <mesh filename="$(find humanoid_robot)/meshes/Foot_Right.STL" />
-            </geometry>
-        </visual>
-        <!-- <collision>
-            <origin xyz="0 0 0" rpy="0 0 0" />
-            <geometry>
-                <mesh filename="$(find humanoid_robot)/meshes/Foot_Right.STL" />
-            </geometry>
-        </collision> -->
+                <mesh filename="file://$(find humanoid_robot)/meshes/Foot_Right.STL" />
+            </geometry>
+        </visual>
+        <collision>
+            <origin xyz="0 0 0" rpy="0 0 0" />
+            <geometry>
+                <mesh filename="file://$(find humanoid_robot)/meshes/Foot_Right.STL" />
+            </geometry>
+        </collision>
         </link>
         <!-- ****************************   Joints   **************************** -->
@@ -391,4 +429,9 @@
             <dynamics damping="0.15" friction="0.2"/>
         </joint>
+        <joint name="ElbowPalm_Left" type="fixed">
+            <origin xyz="0.03 -0.003 -0.14" rpy="0 0 0" />
+            <parent link="Elbow_Left" />
+            <child link="Palm_Left" />
+        </joint>
         <joint name="TorsoShoulder_Right_Roll" type="revolute">
             <origin xyz="-0.033308 0.08489 0.77914" rpy="0 0 0" />
@@ -414,4 +457,9 @@
             <limit lower="-1.74533" upper="0.349066" effort="1.0" velocity="1.0"/> <!-- (-20) to 100 deg-->
             <dynamics damping="0.15" friction="0.2"/>
+        </joint>
+        <joint name="ElbowPalm_Right" type="fixed">
+            <origin xyz="0.03 0.003 -0.14" rpy="0 0 0" />
+            <parent link="Elbow_Right" />
+            <child link="Palm_Right" />
         </joint>
         <joint name="TorsoThigh_Left_Yaw" type="revolute">
